File: bioreactor final/Proyecto_bioreactor.kicad_pcb (KiCad board)
At the start: 2 copper layers, 100 x 60 mm, 38 parts, among them J1 Screw_Terminal_01x02, Q1 IRLZ44N, Q2 NPN, U2 OKI-78SR-5/1.5-W36-C (L7805)

Commit message: Entrega trabajo
Other:
- board text added: "Biorreactor Grupo 7"
Changed lines of the file:
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@@
 			(outputformat 1)
 			(mirror no)
-			(drillshape 1)
+			(drillshape 0)
 			(scaleselection 1)
 			(outputdirectory "")
@@
 		(layer "Edge.Cuts")
 	)
+	(gr_text "Biorreactor Grupo 7"
+		(at 83 108 0)
+		(layer "F.SilkS")
+		(effects
+			(font
+				(size 1 1)
+				(thickness 0.15)
+			)
+		)
+	)
 	(segment
 		(start 80 85.1)
@@
 	)
 	(segment
-		(start 162.05 62.45)
-		(end 160.4 60.8)
-		(width 0.8)
-		(layer "B.Cu")
-		(net "/ALARM-")
-	)
-	(segment
-		(start 154.755 66.015)
-		(end 158.485 66.015)
-		(width 0.8)
-		(layer "B.Cu")
-		(net "/ALARM-")
-	)
-	(segment
-		(start 158.485 66.015)
-		(end 162.05 62.45)
-		(width 0.8)
-		(layer "B.Cu")
-		(net "/ALARM-")
-	)
-	(segment
-		(start 165.5 65.08)
-		(end 164.68 65.08)
-		(width 0.8)
-		(layer "B.Cu")
-		(net "/ALARM-")
-	)
-	(segment
-		(start 164.68 65.08)
-		(end 162.05 62.45)
-		(width 0.8)
-		(layer "B.Cu")
-		(net "/ALARM-")
-	)
-	(segment
 		(start 90.178428 91.55)
 		(end 95.7 86.028428)
@@
 	)
 	(segment
+		(start 162.05 62.45)
+		(end 160.4 60.8)
+		(width 0.8)
+		(layer "B.Cu")
+		(net "/ALARM-")
+	)
+	(segment
+		(start 154.755 66.015)
+		(end 158.485 66.015)
+		(width 0.8)
+		(layer "B.Cu")
+		(net "/ALARM-")
+	)
+	(segment
+		(start 158.485 66.015)
+		(end 162.05 62.45)
+		(width 0.8)
+		(layer "B.Cu")
+		(net "/ALARM-")
+	)
+	(segment
+		(start 165.5 65.08)
+		(end 164.68 65.08)
+		(width 0.8)
+		(layer "B.Cu")
+		(net "/ALARM-")
+	)
+	(segment
+		(start 164.68 65.08)
+		(end 162.05 62.45)
+		(width 0.8)
+		(layer "B.Cu")
+		(net "/ALARM-")
+	)
+	(segment
